File: Hardware/V1/M0 DC Closed Loop Servo.brd (EAGLE design)
At the start: 43.9 x 44.1 mm, 59 parts, among them Q1 2N7002PW, Q2 2.5A/30V, U1 DRV8871, U2 DRV8871, U3 ATSAMD21G-A, U4 3.3V, U5 74AHC1G125, U6 24LC256, Y1 32.768kHz

Commit message: Board Redesign, Rework, and Overhaul to V2
Board Redesign, Rework, and Overhaul to V2
Parts:
- removed ENCDAT, ENCPOW: (no value), SparkFun-Connectors:1X02
- added ENCODER: (no value), SparkFun-Connectors:JST-4-PTH-VERT
- moved R7 30.9 mm to (2.54, 21.6), turned to 0 degrees
- moved Q2 30.6 mm to (2.54, 24.6), turned to 0 degrees
- moved R15 28.3 mm to (30.5, 15.2), turned to 90 degrees
- moved R20 10.9 mm to (23.8, 16.0)
- moved U$8 8.11 mm to (3.89, 41.4)
- moved R18 8.08 mm to (9.45, 21.2)
- moved U$7 6.80 mm to (39.8, 3.43)
- moved D4 6.55 mm to (25.4, 34.3)
- moved R9 6.10 mm to (12.9, 22.4)
- moved R4 5.79 mm to (5.54, 25.9), turned to 270 degrees
- moved SJ1 5.76 mm to (2.01, 29.4), turned to 180 degrees
- moved C2 5.53 mm to (11.4, 16.5)
- moved R14 5.29 mm to (22.9, 19.1), turned to 0 degrees
- moved C9 4.46 mm to (6.35, 22.9), turned to 0 degrees
- moved R21 4.41 mm to (26.5, 16.0)
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Connections:
- net ENCODER: now also ENCODER.3; no longer ENCDAT.1
- net GND: now also ENCODER.1; no longer ENCPOW.1
- net MVIN: now also ENCODER.2; no longer ENCPOW.2
- net N$18: now also ENCODER.4; no longer ENCDAT.2
Routing:
- net 3.3V: track 98.1 -> 152.2 mm, vias 4 -> 5
- net GND: track 270.9 -> 320.1 mm, vias 7 -> 6
- net VIN: track 52.8 -> 97.1 mm, vias 2 -> 5
- net D2: track 35.8 -> 3.91 mm, vias 2 -> 0
- net N$9: track 7.05 -> 36.4 mm, vias 0 -> 2
- net ENCODER: track 8.97 -> 35.8 mm, vias 1 -> 2
- net MVIN: track 92.6 -> 113.2 mm, vias 3 -> 5
- net N$12: track 0.00 -> 17.1 mm, vias 0 -> 2
- net N$18: track 24.7 -> 39.0 mm
- net N$6: track 26.9 -> 39.7 mm
- net N$3: track 23.2 -> 11.6 mm, vias 0 -> 2
- net D4: track 8.14 -> 1.83 mm
- net !RESET: track 27.7 -> 33.7 mm, vias 2 -> 3
- net N$15: track 35.1 -> 29.3 mm, vias 3 -> 2
- net VDDCORE: track 18.6 -> 13.0 mm, vias 0 -> 2
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