File: Hardware/V1/M0 DC Closed Loop Servo.sch (EAGLE design)
At the start: 57 parts, among them Q1 2N7002PW, Q2 2.5A/30V, U1 DRV8871, U2 DRV8871, U3 ATSAMD21G-A, U4 3.3V, U5 74AHC1G125, U6 24LC256, Y1 32.768kHz

Commit message: Board Redesign, Rework, and Overhaul to V2
Board Redesign, Rework, and Overhaul to V2
Parts:
- removed ENCDAT, ENCPOW: (no value), SparkFun-Connectors:CONN_02
- added ENCODER: (no value), SparkFun-Connectors:CONN_04JST-PTH-VERT
Connections:
- net ENCODER: now also ENCODER.3; no longer ENCDAT.1
- net GND: now also ENCODER.1; no longer ENCPOW.1
- net MVIN: now also ENCODER.2; no longer ENCPOW.2
- net N$18: now also ENCODER.4; no longer ENCDAT.2
Changed lines of the file:
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@@
 <?xml version="1.0" encoding="utf-8"?>
 <!DOCTYPE eagle SYSTEM "eagle.dtd">
-<eagle version="8.4.3">
+<eagle version="8.0.0">
 <drawing>
 <settings>
 <setting alwaysvectorfont="no"/>
-<setting keepoldvectorfont="yes"/>
 <setting verticaltext="up"/>
 </settings>
@@
 <part name="SUPPLY19" library="SparkFun-Aesthetics" deviceset="VIN" device=""/>
 <part name="SUPPLY20" library="SparkFun-Aesthetics" deviceset="VIN" device=""/>
+<part name="ENCODER" library="SparkFun-Connectors" deviceset="CONN_04" device="JST-PTH-VERT"/>
 <part name="AUX" library="SparkFun-Connectors" deviceset="CONN_03" device="LONGPADS"/>
 <part name="R11" library="SparkFun-Resistors" deviceset="1KOHM" device="-0603-1/10W-1%" value="1k"/>
@@
 <part name="R20" library="SparkFun-Resistors" deviceset="10KOHM" device="-0603-1/10W-1%" value="10k"/>
 <part name="R21" library="SparkFun-Resistors" deviceset="10KOHM" device="-0603-1/10W-1%" value="10k"/>
-<part name="ENCDAT" library="SparkFun-Connectors" deviceset="CONN_02" device=""/>
-<part name="ENCPOW" library="SparkFun-Connectors" deviceset="CONN_02" device=""/>
 </parts>
 <sheets>
@@
 <instance part="SUPPLY19" gate="G$1" x="94.488" y="173.228"/>
 <instance part="SUPPLY20" gate="G$1" x="208.788" y="74.168"/>
+<instance part="ENCODER" gate="G$1" x="144.78" y="22.86"/>
 <instance part="AUX" gate="J$1" x="142.24" y="39.624"/>
 <instance part="R11" gate="G$1" x="143.764" y="52.324"/>
@@
 <instance part="R20" gate="G$1" x="231.14" y="71.12"/>
 <instance part="R21" gate="G$1" x="246.38" y="71.12"/>
-<instance part="ENCDAT" gate="G$1" x="142.24" y="25.4"/>
-<instance part="ENCPOW" gate="G$1" x="132.08" y="17.78"/>
 </instances>
 <busses>
@@
 <wire x1="178.308" y1="20.32" x2="178.308" y2="41.148" width="0.1524" layer="91"/>
 <junction x="178.308" y="41.148"/>
-<wire x1="139.7" y1="17.78" x2="178.308" y2="20.32" width="0.1524" layer="91"/>
-<pinref part="ENCPOW" gate="G$1" pin="1"/>
+<pinref part="ENCODER" gate="G$1" pin="1"/>
+<wire x1="149.86" y1="20.32" x2="178.308" y2="20.32" width="0.1524" layer="91"/>
 </segment>
 <segment>
@@
 </segment>
 <segment>
+<pinref part="C2" gate="G$1" pin="-"/>
 <pinref part="U$2" gate="G$1" pin="GND"/>
-<pinref part="C2" gate="G$1" pin="-"/>
 <wire x1="193.548" y1="-14.732" x2="193.548" y2="-17.272" width="0.1524" layer="91"/>
+<pinref part="IN" gate="G$1" pin="2"/>
+<wire x1="207.264" y1="-2.032" x2="206.248" y2="-17.272" width="0.1524" layer="91"/>
+<wire x1="206.248" y1="-17.272" x2="193.548" y2="-17.272" width="0.1524" layer="91"/>
+<junction x="193.548" y="-17.272"/>
+<wire x1="207.264" y1="-2.54" x2="207.264" y2="-2.032" width="0.1524" layer="91"/>
+<junction x="207.264" y="-2.032"/>
 <pinref part="NJM78L00UA" gate="G$1" pin="GND"/>
-<wire x1="223.52" y1="-7.62" x2="208.28" y2="-7.62" width="0.1524" layer="91"/>
-<wire x1="207.264" y1="-7.62" x2="198.12" y2="-7.62" width="0.1524" layer="91"/>
-<wire x1="198.12" y1="-7.62" x2="198.12" y2="-20.32" width="0.1524" layer="91"/>
-<wire x1="198.12" y1="-20.32" x2="193.548" y2="-20.32" width="0.1524" layer="91"/>
-<wire x1="193.548" y1="-20.32" x2="193.548" y2="-17.272" width="0.1524" layer="91"/>
-<junction x="193.548" y="-17.272"/>
-<pinref part="IN" gate="G$1" pin="2"/>
-<wire x1="207.264" y1="-2.54" x2="207.264" y2="-2.032" width="0.1524" layer="91"/>
-<wire x1="208.28" y1="-7.62" x2="207.264" y2="-7.62" width="0.1524" layer="91"/>
+<wire x1="223.52" y1="-7.62" x2="207.264" y2="-7.62" width="0.1524" layer="91"/>
 <wire x1="207.264" y1="-7.62" x2="207.264" y2="-2.032" width="0.1524" layer="91"/>
-<junction x="207.264" y="-2.032"/>
 </segment>
 <segment>
@@
 <wire x1="138.684" y1="72.136" x2="134.874" y2="72.136" width="0.1524" layer="91"/>
 <wire x1="134.874" y1="72.136" x2="134.874" y2="28.956" width="0.1524" layer="91"/>
+<pinref part="ENCODER" gate="G$1" pin="4"/>
 <wire x1="134.874" y1="28.956" x2="149.86" y2="28.956" width="0.1524" layer="91"/>
 <wire x1="149.86" y1="28.956" x2="149.86" y2="27.94" width="0.1524" layer="91"/>
@@
 <wire x1="138.684" y1="75.438" x2="138.684" y2="72.136" width="0.1524" layer="91"/>
 <junction x="138.684" y="72.136"/>
-<pinref part="ENCDAT" gate="G$1" pin="2"/>
 </segment>
 </net>
@@
 <wire x1="139.192" y1="78.74" x2="133.858" y2="78.74" width="0.1524" layer="91"/>
 <wire x1="133.858" y1="78.74" x2="133.858" y2="26.67" width="0.1524" layer="91"/>
+<pinref part="ENCODER" gate="G$1" pin="3"/>
 <wire x1="133.858" y1="26.67" x2="149.86" y2="26.67" width="0.1524" layer="91"/>
 <wire x1="149.86" y1="26.67" x2="149.86" y2="25.4" width="0.1524" layer="91"/>
@@
 <wire x1="139.192" y1="82.55" x2="139.192" y2="78.74" width="0.1524" layer="91"/>
 <junction x="139.192" y="78.74"/>
-<pinref part="ENCDAT" gate="G$1" pin="1"/>
 </segment>
 </net>
@@
 <junction x="193.548" y="-2.032"/>
 <pinref part="IN" gate="G$1" pin="1"/>
+<pinref part="NJM78L00UA" gate="G$1" pin="IN"/>
+<wire x1="223.52" y1="0" x2="204.724" y2="0" width="0.1524" layer="91"/>
 <wire x1="204.724" y1="0" x2="204.724" y2="-2.032" width="0.1524" layer="91"/>
 <junction x="204.724" y="-2.032"/>
@@
 <wire x1="180.34" y1="-5.08" x2="147.828" y2="-5.08" width="0.1524" layer="91"/>
 <wire x1="147.828" y1="-5.08" x2="147.828" y2="-2.032" width="0.1524" layer="91"/>
-<pinref part="NJM78L00UA" gate="G$1" pin="IN"/>
-<wire x1="223.52" y1="0" x2="213.36" y2="0" width="0.1524" layer="91"/>
-<wire x1="213.36" y1="0" x2="213.36" y2="12.7" width="0.1524" layer="91"/>
-<wire x1="213.36" y1="12.7" x2="204.724" y2="12.7" width="0.1524" layer="91"/>
-<wire x1="204.724" y1="12.7" x2="204.724" y2="-2.032" width="0.1524" layer="91"/>
-</segment>
-<segment>
+</segment>
+<segment>
+<pinref part="ENCODER" gate="G$1" pin="2"/>
 <wire x1="155.448" y1="22.352" x2="150.368" y2="22.352" width="0.1524" layer="91"/>
-<wire x1="150.368" y1="22.352" x2="139.7" y2="20.32" width="0.1524" layer="91"/>
+<wire x1="150.368" y1="22.352" x2="149.86" y2="22.86" width="0.1524" layer="91"/>
 <label x="152.4" y="22.86" size="1.778" layer="95"/>
-<pinref part="ENCPOW" gate="G$1" pin="2"/>
-</segment>
-</net>
+</segment>
+</net>
