File: Hardware/M0 DC Closed Loop Servo.sch (EAGLE design)
At the start: 57 parts, among them Q1 2N7002PW, Q2 2.5A/30V, U1 DRV8871, U2 DRV8871, U3 ATSAMD21G-A, U4 3.3V, U5 74AHC1G125, U6 24LC256, Y1 32.768kHz

Commit message: Board Clean UP
Parts:
- removed SJ1: PWR-LED, SparkFun-Passives:JUMPER-PAD-2-NC_BY_TRACENO_SILK
- NJM: value AP1117Y33G-13 -> NJM78L00UA
- U6: value 24LC256 -> EEPROM-I2CSMD
- renumbered NJM78L00UA to NJM
Connections:
- net GND: no longer SJ1.1
- net N$12: no longer SJ1.2
Changed lines of the file:
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@@
 <part name="R8" library="SparkFun-Resistors" deviceset="330OHM1/10W1%(0603)" device="" value="330"/>
 <part name="SUPPLY16" library="SparkFun-Aesthetics" deviceset="3.3V" device=""/>
-<part name="SJ1" library="SparkFun-Passives" deviceset="JUMPER-PAD-2-NC_BY_TRACE" device="NO_SILK" value="PWR-LED"/>
 <part name="S1" library="samd21-temp" deviceset="SWITCH-MOMENTARY-2" device="SMD-4.6X2.8MM" value="RESET"/>
 <part name="SUPPLY17" library="SparkFun-Aesthetics" deviceset="VIN" device=""/>
@@
 <part name="OUT" library="SparkFun-Connectors" deviceset="CONN_02" device="PTH3"/>
 <part name="IN" library="SparkFun-Connectors" deviceset="CONN_02" device="PTH3"/>
-<part name="NJM78L00UA" library="AP1117Y33G-13" deviceset="AP1117Y33G-13" device=""/>
+<part name="NJM" library="AP1117Y33G-13" deviceset="AP1117Y33G-13" device="" value="NJM78L00UA"/>
 <part name="CN1" library="adafruit" deviceset="USB" device="MINIB"/>
 <part name="U2" library="microbuilder" deviceset="DRV8871" device="" value="DRV8871"/>
-<part name="U6" library="SparkFun-IC-Memory" deviceset="EEPROM-I2C" device="SMD" value="24LC256"/>
+<part name="U6" library="SparkFun-IC-Memory" deviceset="EEPROM-I2C" device="SMD" value="EEPROM-I2CSMD"/>
 <part name="R20" library="SparkFun-Resistors" deviceset="10KOHM" device="-0603-1/10W-1%" value="10k"/>
 <part name="R21" library="SparkFun-Resistors" deviceset="10KOHM" device="-0603-1/10W-1%" value="10k"/>
@@
 <instance part="R3" gate="G$1" x="160.528" y="160.528" rot="R90"/>
 <instance part="SUPPLY11" gate="G$1" x="211.328" y="168.148"/>
-<instance part="GND14" gate="1" x="211.328" y="127.508"/>
+<instance part="GND14" gate="1" x="211.328" y="137.668"/>
 <instance part="GND15" gate="1" x="160.528" y="127.508"/>
 <instance part="D3" gate="G$1" x="160.528" y="150.368"/>
@@
 <instance part="R8" gate="G$1" x="193.548" y="160.528" rot="R90"/>
 <instance part="SUPPLY16" gate="G$1" x="193.548" y="168.148"/>
-<instance part="SJ1" gate="G$1" x="211.328" y="137.668" rot="MR90"/>
 <instance part="S1" gate="G$1" x="4.064" y="22.098" rot="MR0"/>
 <instance part="SUPPLY17" gate="G$1" x="43.688" y="150.368"/>
@@
 <instance part="OUT" gate="G$1" x="196.088" y="15.24" rot="R270"/>
 <instance part="IN" gate="G$1" x="204.724" y="5.588" rot="R270"/>
-<instance part="NJM78L00UA" gate="G$1" x="228.6" y="-10.16"/>
+<instance part="NJM" gate="G$1" x="228.6" y="-10.16"/>
 <instance part="CN1" gate="G$1" x="7.62" y="162.56"/>
 <instance part="U2" gate="G$1" x="135.128" y="0.508"/>
@@
 <segment>
 <pinref part="GND14" gate="1" pin="GND"/>
-<pinref part="SJ1" gate="G$1" pin="1"/>
-<wire x1="211.328" y1="132.588" x2="211.328" y2="130.048" width="0.1524" layer="91"/>
+<wire x1="211.328" y1="145.288" x2="211.328" y2="140.208" width="0.1524" layer="91"/>
 </segment>
 <segment>
@@
 <pinref part="C2" gate="G$1" pin="-"/>
 <wire x1="193.548" y1="-14.732" x2="193.548" y2="-17.272" width="0.1524" layer="91"/>
-<pinref part="NJM78L00UA" gate="G$1" pin="GND"/>
+<pinref part="NJM" gate="G$1" pin="GND"/>
 <wire x1="223.52" y1="-7.62" x2="208.28" y2="-7.62" width="0.1524" layer="91"/>
 <wire x1="207.264" y1="-7.62" x2="198.12" y2="-7.62" width="0.1524" layer="91"/>
@@
 <wire x1="193.04" y1="74.168" x2="193.04" y2="27.94" width="0.1524" layer="91"/>
 <junction x="206.248" y="74.168"/>
-<pinref part="NJM78L00UA" gate="G$1" pin="OUT"/>
+<pinref part="NJM" gate="G$1" pin="OUT"/>
 <wire x1="193.04" y1="27.94" x2="246.38" y2="27.94" width="0.1524" layer="91"/>
 <wire x1="246.38" y1="27.94" x2="246.38" y2="0" width="0.1524" layer="91"/>
@@
 <segment>
 <pinref part="D2" gate="G$1" pin="C"/>
-<pinref part="SJ1" gate="G$1" pin="2"/>
 <wire x1="211.328" y1="142.748" x2="211.328" y2="145.288" width="0.1524" layer="91"/>
 </segment>
@@
 <wire x1="180.34" y1="-5.08" x2="147.828" y2="-5.08" width="0.1524" layer="91"/>
 <wire x1="147.828" y1="-5.08" x2="147.828" y2="-2.032" width="0.1524" layer="91"/>
-<pinref part="NJM78L00UA" gate="G$1" pin="IN"/>
+<pinref part="NJM" gate="G$1" pin="IN"/>
 <wire x1="223.52" y1="0" x2="213.36" y2="0" width="0.1524" layer="91"/>
 <wire x1="213.36" y1="0" x2="213.36" y2="12.7" width="0.1524" layer="91"/>

Commit message: COMPLETE OVER HULL
Parts:
- removed R10, R16, R17, R18, R9: 2.0k, SparkFun-Resistors:2.0KOHM-0603-1/10W-5%
- removed R11, R12, R13, R14, R15: 1k, SparkFun-Resistors:1KOHM-0603-1/10W-1%
- added J1: (no value), SparkFun-Connectors:CONN_02
Connections:
- removed net ENCODER: ENCDAT.1, R15.1, R18.2
- removed net N$14: AUX.3, R11.1, R17.2
- removed net N$16: AUX.2, R12.1, R9.2
- removed net N$17: AUX.1, R10.2, R13.1
- removed net N$18: ENCDAT.2, R14.1, R16.2
- net D0/RXI: now also J1.1
- net D1/TXO: now also J1.2
- net D2: now also ENCDAT.2; no longer R15.2
- net D3: now also AUX.3
- net D4: now also ENCDAT.1; no longer R14.2
- net D7: no longer R13.2
- net D8: now also AUX.2; no longer R12.2
- net D9: now also AUX.1; no longer R11.2
- net GND: no longer R10.1, R16.1, R17.1, R18.1, R9.1
Other:
- moved on the sheet: AUX, C1, C2, ENCDAT, ENCPOW, I2C, IN, NJM, OUT, R19, R20, R21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
