File: Hardware/M0 DC Closed Loop Servo.brd (EAGLE design)
At the start: 43.9 x 44.1 mm, 59 parts, among them Q1 2N7002PW, Q2 2.5A/30V, U1 DRV8871, U2 DRV8871, U3 ATSAMD21G-A, U4 3.3V, U5 74AHC1G125, U6 24LC256, Y1 32.768kHz

Commit message: Board Clean UP
Parts:
- removed SJ1: PWR-LED, SparkFun-Passives:PAD-JUMPER-2-NC_BY_TRACE_NO_SILK
- NJM: value AP1117Y33G-13 -> NJM78L00UA
- U6: value 24LC256 -> EEPROM-I2CSMD
- moved D2 12.0 mm to (27.3, 33.7)
- moved D3 8.87 mm to (25.5, 33.7)
- moved D4 2.74 mm to (29.2, 33.7)
- moved D1 2.10 mm to (31.0, 33.7)
- moved I2C 0.25 mm to (33.0, 2.29)
- moved JP5 0.25 mm to (28.1, 30.2)
- renumbered NJM78L00UA to NJM
Connections:
- net GND: no longer SJ1.1
- net N$12: no longer SJ1.2
Routing:
- net N$5: track 1.44 -> 51.5 mm, vias 0 -> 4
- net N$3: track 23.2 -> 38.3 mm
- net RX_LED: track 0.00 -> 9.57 mm
- net 3.3V: track 98.1 -> 106.4 mm
- net N$6: track 26.9 -> 21.3 mm, vias 2 -> 4
- net N$11: track 0.00 -> 4.91 mm
- net SWCLK: track 14.9 -> 10.4 mm
- net VIN: track 52.8 -> 57.0 mm, vias 2 -> 3
- net !RESET: track 27.7 -> 24.7 mm, vias 2 -> 1
- net GND: track 270.9 -> 273.1 mm, vias 7 -> 9
- net N$17: track 29.2 -> 30.4 mm, vias 1 -> 4
- net TX_LED: track 6.78 -> 7.52 mm

Commit message: COMPLETE OVER HULL
Parts:
- removed R10, R16, R17, R18, R9: 2.0k, SparkFun-Resistors:0603
- removed R11, R12, R13, R14, R15: 1k, SparkFun-Resistors:0603
- added J1: (no value), SparkFun-Connectors:1X02
Connections:
- removed net ENCODER: ENCDAT.1, R15.1, R18.2
- removed net N$14: AUX.3, R11.1, R17.2
- removed net N$16: AUX.2, R12.1, R9.2
- removed net N$17: AUX.1, R10.2, R13.1
- removed net N$18: ENCDAT.2, R14.1, R16.2
- net D0/RXI: now also J1.1
- net D1/TXO: now also J1.2
- net D2: now also ENCDAT.2; no longer R15.2
- net D3: now also AUX.3
- net D4: now also ENCDAT.1; no longer R14.2
- net D7: no longer R13.2
- net D8: now also AUX.2; no longer R12.2
- net D9: now also AUX.1; no longer R11.2
- net GND: no longer R10.1, R16.1, R17.1, R18.1, R9.1
Routing:
- net D8: track 4.23 -> 34.7 mm, vias 0 -> 2
- net D3: track 0.00 -> 30.4 mm, vias 0 -> 2
- net N$17: track 30.4 -> 0.00 mm, vias 4 -> 0
- net N$16: track 28.4 -> 0.00 mm, vias 3 -> 0
- net D4: track 8.14 -> 33.8 mm, vias 0 -> 1
- net N$18: track 24.7 -> 0.00 mm, vias 1 -> 0
- net N$14: track 24.1 -> 0.00 mm
- net D9: track 3.89 -> 26.5 mm
- net D0/RXI: track 0.00 -> 20.2 mm, vias 0 -> 3
- net D1/TXO: track 0.00 -> 19.2 mm, vias 0 -> 3
- net D2: track 35.8 -> 45.2 mm, vias 2 -> 3
- net ENCODER: track 8.97 -> 0.00 mm, vias 1 -> 0
- net GND: track 273.1 -> 265.5 mm, vias 9 -> 10
- net D7: track 6.96 -> 9.34 mm
- net SDA: track 29.2 -> 27.0 mm
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Other:
- board text added: "TX RX"

Commit message: rey-load
Parts:
- moved U$7 0.80 mm to (36.7, 9.58)
Routing:
- net D7: track 9.34 -> 0.00 mm
- net D2: track 45.2 -> 37.2 mm
Changed lines of the file:
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@@
 <attribute name="PROD_ID" value="XTAL-13062" x="21.082" y="28.6004" size="1.778" layer="27" display="off"/>
 </element>
-<element name="U$7" library="fiducial" package="CIRCLE-1MM-3R" value="" x="37.4904" y="9.8298"/>
+<element name="U$7" library="fiducial" package="CIRCLE-1MM-3R" value="" x="36.7284" y="9.5758"/>
 <element name="U$8" library="fiducial" package="CIRCLE-1MM-3R" value="" x="9.144" y="35.2044"/>
 <element name="NJM" library="AP1117Y33G-13" package="SOT89" value="NJM78L00UA" x="41.148" y="9.144" rot="R180"/>
@@
 <signal name="D2">
 <contactref element="U3" pad="23"/>
-<wire x1="7.9248" y1="24.9301" x2="4.7879" y2="24.9301" width="0.127" layer="1"/>
-<wire x1="8.9154" y1="24.9301" x2="7.9248" y2="24.9301" width="0.127" layer="16"/>
-<wire x1="13.5382" y1="29.5529" x2="8.9154" y2="24.9301" width="0.127" layer="16"/>
-<wire x1="14.5288" y1="29.5529" x2="13.5382" y2="29.5529" width="0.127" layer="16"/>
-<wire x1="21.6281" y1="22.4536" x2="14.5288" y2="29.5529" width="0.127" layer="16"/>
-<wire x1="27.4066" y1="22.4536" x2="21.6281" y2="22.4536" width="0.127" layer="16"/>
-<wire x1="28.8925" y1="23.9395" x2="27.4066" y2="22.4536" width="0.127" layer="16"/>
-<wire x1="28.8925" y1="24.1046" x2="28.8925" y2="23.9395" width="0.127" layer="16"/>
-<wire x1="28.8925" y1="20.8026" x2="28.8925" y2="24.1046" width="0.127" layer="1"/>
-<wire x1="30.2133" y1="19.4818" x2="28.8925" y2="20.8026" width="0.127" layer="1"/>
-<wire x1="30.2133" y1="18.8214" x2="30.2133" y2="19.4818" width="0.127" layer="1"/>
+<contactref element="ENCDAT" pad="2"/>
+<wire x1="30.2133" y1="19.4818" x2="30.2133" y2="18.8214" width="0.127" layer="1"/>
+<wire x1="29.3878" y1="20.3073" x2="30.2133" y2="19.4818" width="0.127" layer="1"/>
+<wire x1="27.4066" y1="20.3073" x2="29.3878" y2="20.3073" width="0.127" layer="16"/>
+<wire x1="20.4724" y1="13.3731" x2="27.4066" y2="20.3073" width="0.127" layer="16"/>
+<wire x1="20.4724" y1="14.0335" x2="20.4724" y2="13.3731" width="0.127" layer="1"/>
+<wire x1="17.1704" y1="17.3355" x2="20.4724" y2="14.0335" width="0.127" layer="1"/>
+<wire x1="17.1704" y1="18.8214" x2="17.1704" y2="17.3355" width="0.127" layer="1"/>
+<wire x1="16.6751" y1="19.3167" x2="17.1704" y2="18.8214" width="0.127" layer="1"/>
+<wire x1="11.8872" y1="19.3167" x2="16.6751" y2="19.3167" width="0.127" layer="1"/>
+<wire x1="4.6228" y1="19.3167" x2="11.8872" y2="19.3167" width="0.127" layer="16"/>
+<wire x1="1.9812" y1="16.6751" x2="4.6228" y2="19.3167" width="0.127" layer="16"/>
 <wire x1="30.2133" y1="18.8214" x2="30.19" y2="18.737" width="0.127" layer="1"/>
-<via x="7.9248" y="24.9301" extent="1-16" drill="0.6096"/>
-<via x="28.8925" y="24.1046" extent="1-16" drill="0.6096"/>
-<contactref element="ENCDAT" pad="2"/>
-<wire x1="1.9812" y1="17.5006" x2="1.9812" y2="16.6751" width="0.127" layer="16"/>
-<wire x1="4.7879" y1="20.3073" x2="1.9812" y2="17.5006" width="0.127" layer="16"/>
-<wire x1="4.7879" y1="24.9301" x2="4.7879" y2="20.3073" width="0.127" layer="16"/>
 <wire x1="1.9812" y1="16.6751" x2="1.8288" y2="16.6624" width="0.127" layer="16"/>
-<via x="4.7879" y="24.9301" extent="1-16" drill="0.6096"/>
+<via x="29.3878" y="20.3073" extent="1-16" drill="0.6096"/>
+<via x="20.4724" y="13.3731" extent="1-16" drill="0.6096"/>
+<via x="11.8872" y="19.3167" extent="1-16" drill="0.6096"/>
 </signal>
 <signal name="D5">
@@
 <signal name="D7">
 <contactref element="U3" pad="30"/>
-<wire x1="37.4777" y1="22.7838" x2="38.4683" y2="22.7838" width="0.127" layer="1"/>
-<wire x1="36.8173" y1="22.1234" x2="37.4777" y2="22.7838" width="0.127" layer="1"/>
-<wire x1="33.6804" y1="22.1234" x2="34.671" y2="22.1234" width="0.127" layer="1"/>
-<wire x1="34.671" y1="22.1234" x2="36.8173" y2="22.1234" width="0.127" layer="1"/>
-<wire x1="33.02" y1="22.7838" x2="33.6804" y2="22.1234" width="0.127" layer="1"/>
-<wire x1="32.1945" y1="22.7838" x2="33.02" y2="22.7838" width="0.127" layer="1"/>
-<wire x1="32.1945" y1="22.7838" x2="32.19" y2="22.737" width="0.127" layer="1"/>
-<wire x1="34.671" y1="22.1234" x2="34.671" y2="24.5999" width="0.127" layer="1"/>
 </signal>
 <signal name="D8">
